Commit message: Start migrating to Ros Humble with Ubuntu 22.04

File: yahboom_rosmaster_description/urdf/control/rosmaster_x3_ros2_control.urdf.xacro (robot description, xacro)
@@ -4,7 +4,5 @@
         <ros2_control name="RobotSystem" type="system">
             <hardware>
-                <xacro:if value="${use_gazebo}">
-                    <plugin>gz_ros2_control/GazeboSimSystem</plugin>
-                </xacro:if>
+                <plugin>gazebo_ros2_control/GazeboSystem</plugin>
             </hardware>
             <joint name="${prefix}front_left_wheel_joint">

File: yahboom_rosmaster_description/urdf/mech/mecanum_wheel.urdf.xacro (robot description, xacro)
@@ -4,5 +4,5 @@
   <xacro:property name="wheel_separation" value="0.169" />
   <xacro:property name="wheel_width" value="0.03040" />
-  <xacro:property name="wheel_mass" value="9.1" />
+  <xacro:property name="wheel_mass" value="0.4" />
   <xacro:property name="wheel_xoff" value="0.08" />
   <xacro:property name="wheel_yoff" value="-0.01" />
@@ -21,5 +21,5 @@
         <origin xyz="0 0 0" rpy="${pi/2} 0 0"/>
         <geometry>
-          <cylinder radius="${wheel_radius}" length="${wheel_width}"/>
+          <sphere radius="${wheel_radius}"/>
         </geometry>
       </collision>
@@ -37,24 +37,42 @@
       <parent link="${prefix}base_link"/>
       <child link="${prefix}${side}_wheel_link"/>
-      <origin xyz="${x_reflect*wheel_xoff} ${y_reflect*(wheel_separation/2+wheel_yoff)} ${-wheel_radius}" rpy="0 0 0"/>
+      <origin xyz="${x_reflect*wheel_xoff} ${y_reflect*(wheel_separation/2+wheel_yoff)} -0.003" rpy="0 0 0"/>
+      <limit effort="10.0" velocity="10.0"/>
     </joint>
+    <!-- Add joint damping/friction to reduce drift at rest -->
+    <gazebo reference="${prefix}${side}_wheel_joint">
+      <dynamics damping="0.01" friction="0.0"/>
+    </gazebo>
+    <!-- Wheel contact/friction tuning for Gazebo Classic -->
+    <!-- Wheel contact/friction tuning for Gazebo Classic -->
     <gazebo reference="${prefix}${side}_wheel_link">
       <surface>
         <friction>
           <ode>
-              <mu>1.0</mu>
-              <mu2>0.0</mu2>
+            <mu>0.8</mu>
+            <mu2>0.8</mu2>
+            <fdir1>1 0 0</fdir1>
+            <slip1>0.0</slip1>
+            <slip2>0.0</slip2>
           </ode>
         </friction>
+        <contact>
+          <ode>
+            <kp>1000000.0</kp>
+            <kd>100.0</kd>
+            <max_vel>0.1</max_vel>
+            <min_depth>0.001</min_depth>
+          </ode>
+        </contact>
       </surface>
       <visual>
-          <material>
-              <ambient>0.2 0.2 0.2 1.0</ambient>
-              <diffuse>0.2 0.2 0.2 1.0</diffuse>
-              <specular>0.2 0.2 0.2 1.0</specular>
-              <emissive>0.0 0.0 0.0 0.0</emissive>
-          </material>
+        <material>
+          <ambient>0.2 0.2 0.2 1.0</ambient>
+          <diffuse>0.2 0.2 0.2 1.0</diffuse>
+          <specular>0.2 0.2 0.2 1.0</specular>
+          <emissive>0.0 0.0 0.0 0.0</emissive>
+        </material>
       </visual>
-  </gazebo>
+    </gazebo>
   </xacro:macro>
 </robot>

File: yahboom_rosmaster_description/urdf/robots/rosmaster_x3.urdf.xacro (robot description, xacro)
@@ -1,65 +1,68 @@
 <?xml version="1.0"?>
 <robot xmlns:xacro="http://www.ros.org/wiki/xacro" name="rosmaster_x3">
-    <xacro:property name="M_PI" value="3.1415926535897931" />
-    <xacro:arg name="robot_name" default="rosmaster_x3"/>
-    <xacro:arg name="prefix" default=""/>
-    <xacro:arg name="use_gazebo" default="false"/>
-    <xacro:include filename="$(find yahboom_rosmaster_description)/urdf/mech/rosmaster_x3_base.urdf.xacro"/>
-    <xacro:include filename="$(find yahboom_rosmaster_description)/urdf/mech/mecanum_wheel.urdf.xacro"/>
-    <xacro:include filename="$(find yahboom_rosmaster_description)/urdf/sensors/rgbd_camera.urdf.xacro"/>
-    <xacro:include filename="$(find yahboom_rosmaster_description)/urdf/sensors/lidar.urdf.xacro"/>
-    <xacro:include filename="$(find yahboom_rosmaster_description)/urdf/sensors/imu.urdf.xacro"/>
-    <xacro:rosmaster_x3_base prefix="$(arg prefix)"/>
-    <xacro:mecanum_wheel
-      prefix="$(arg prefix)"
-      side="front_left"
-      x_reflect="1"
-      y_reflect="1"/>
-    <xacro:mecanum_wheel
-      prefix="$(arg prefix)"
-      side="front_right"
-      x_reflect="1"
-      y_reflect="-1"/>
-    <xacro:mecanum_wheel
-      prefix="$(arg prefix)"
-      side="back_left"
-      x_reflect="-1"
-      y_reflect="1"/>
-    <xacro:mecanum_wheel
-      prefix="$(arg prefix)"
-      side="back_right"
-      x_reflect="-1"
-      y_reflect="-1"/>
-    <xacro:rgbd_camera
-      prefix="$(arg prefix)"
-      camera_name="cam_1"
-      xyz_offset="0.105 0 0.05"
-      rpy_offset="0 -0.50 0"/>
-    <xacro:lidar_sensor
-      prefix="$(arg prefix)"
-      parent="base_link"
-      frame_id="laser_frame"
-      xyz_offset="0 0 0.0825"
-      rpy_offset="0 0 0"
-      mesh_xyz_offset="0 0 0"
-      mesh_rpy_offset="${-M_PI/2} 0 0"
-      topic_name="scan"/>
-    <xacro:imu_sensor
-      prefix="$(arg prefix)"
-      parent="base_link"
-      frame_id="imu"
-      xyz_offset="0 0 0.006"
-      rpy_offset="0 0 0"
-      update_rate="15.0"
-      topic_name="imu/data"/>
-    <xacro:include filename="$(find yahboom_rosmaster_description)/urdf/control/velocity_control_plugin.urdf.xacro" />
-    <xacro:load_velocity_control_plugin use_gazebo="$(arg use_gazebo)"/>
-    <xacro:include filename="$(find yahboom_rosmaster_description)/urdf/control/gazebo_sim_ros2_control.urdf.xacro" />
-    <xacro:load_gazebo_sim_ros2_control_plugin
-      robot_name="$(arg robot_name)"
-      use_gazebo="$(arg use_gazebo)"/>
-    <xacro:include filename="$(find yahboom_rosmaster_description)/urdf/control/rosmaster_x3_ros2_control.urdf.xacro" />
-    <xacro:yahboom_rosmaster_ros2_control
-      prefix="$(arg prefix)"
-      use_gazebo="$(arg use_gazebo)"/>
+  <xacro:property name="M_PI" value="3.1415926535897931" />
+  <xacro:arg name="robot_name" default="rosmaster_x3"/>
+  <xacro:arg name="prefix" default=""/>
+  <xacro:arg name="use_gazebo" default="false"/>
+  <xacro:include filename="$(find yahboom_rosmaster_description)/urdf/mech/rosmaster_x3_base.urdf.xacro"/>
+  <xacro:include filename="$(find yahboom_rosmaster_description)/urdf/mech/mecanum_wheel.urdf.xacro"/>
+  <xacro:include filename="$(find yahboom_rosmaster_description)/urdf/sensors/rgbd_camera.urdf.xacro"/>
+  <xacro:include filename="$(find yahboom_rosmaster_description)/urdf/sensors/lidar.urdf.xacro"/>
+  <xacro:include filename="$(find yahboom_rosmaster_description)/urdf/sensors/imu.urdf.xacro"/>
+  <xacro:rosmaster_x3_base prefix="$(arg prefix)"/>
+  <xacro:mecanum_wheel
+    prefix="$(arg prefix)"
+    side="front_left"
+    x_reflect="1"
+    y_reflect="1"/>
+  <xacro:mecanum_wheel
+    prefix="$(arg prefix)"
+    side="front_right"
+    x_reflect="1"
+    y_reflect="-1"/>
+  <xacro:mecanum_wheel
+    prefix="$(arg prefix)"
+    side="back_left"
+    x_reflect="-1"
+    y_reflect="1"/>
+  <xacro:mecanum_wheel
+    prefix="$(arg prefix)"
+    side="back_right"
+    x_reflect="-1"
+    y_reflect="-1"/>
+  <xacro:rgbd_camera
+    prefix="$(arg prefix)"
+    camera_name="cam_1"
+    xyz_offset="0.105 0 0.05"
+    rpy_offset="0 -0.50 0"/>
+  <xacro:lidar_sensor
+    prefix="$(arg prefix)"
+    parent="base_link"
+    frame_id="laser_frame"
+    xyz_offset="0 0 0.0825"
+    rpy_offset="0 0 0"
+    mesh_xyz_offset="0 0 0"
+    mesh_rpy_offset="${-M_PI/2} 0 0"
+    topic_name="scan"/>
+  <xacro:imu_sensor
+    prefix="$(arg prefix)"
+    parent="base_link"
+    frame_id="imu"
+    xyz_offset="0 0 0.006"
+    rpy_offset="0 0 0"
+    update_rate="15.0"
+    topic_name="imu/data"/>
+  <!-- Gazebo Classic ros2_control plugin -->
+  <xacro:if value="$(arg use_gazebo)">
+    <gazebo>
+      <plugin name="gazebo_ros2_control" filename="libgazebo_ros2_control.so">
+        <parameters>$(find yahboom_rosmaster_gazebo)/config/ros2_control.yaml</parameters>
+      </plugin>
+    </gazebo>
+  </xacro:if>
+  <!-- ros2_control joints/interfaces for the robot -->
+  <xacro:include filename="$(find yahboom_rosmaster_description)/urdf/control/rosmaster_x3_ros2_control.urdf.xacro" />
+  <xacro:yahboom_rosmaster_ros2_control
+    prefix="$(arg prefix)"
+    use_gazebo="$(arg use_gazebo)"/>
 </robot>

File: yahboom_rosmaster_description/urdf/sensors/imu.urdf.xacro (robot description, xacro)
@@ -60,5 +60,11 @@
             </material>
             <sensor name="${prefix}imu_sensor" type="imu">
-                <topic>${topic_name}</topic>
+                <plugin name="${prefix}imu_plugin" filename="libgazebo_ros_imu_sensor.so">
+                    <ros>
+                        <namespace>${prefix}</namespace>
+                        <remapping>~/out:=${topic_name}</remapping>
+                    </ros>
+                    <initial_orientation_as_reference>false</initial_orientation_as_reference>
+                </plugin>
                 <update_rate>${update_rate}</update_rate>
                 <always_on>${always_on}</always_on>

File: yahboom_rosmaster_description/urdf/sensors/lidar.urdf.xacro (robot description, xacro)
@@ -79,6 +79,13 @@
         <specular>${gazebo_material_specular}</specular>
       </material>
-      <sensor name="${prefix}lidar_sensor" type="gpu_lidar">
-        <topic>${topic_name}</topic>
+      <sensor name="${prefix}lidar_sensor" type="ray">
+        <plugin name="${prefix}lidar_plugin" filename="libgazebo_ros_ray_sensor.so">
+          <ros>
+            <namespace>${prefix}</namespace>
+            <remapping>~/out:=${topic_name}</remapping>
+          </ros>
+          <output_type>sensor_msgs/LaserScan</output_type>
+          <frame_name>${prefix}${frame_id}</frame_name>
+        </plugin>
         <update_rate>${update_rate}</update_rate>
         <always_on>${always_on}</always_on>

File: yahboom_rosmaster_description/urdf/sensors/rgbd_camera.urdf.xacro (robot description, xacro)
@@ -125,5 +125,16 @@
     <link name="${prefix}${camera_name}_color_optical_frame"/>
     <gazebo reference="${prefix}${camera_name}_link">
-      <sensor name="${prefix}${camera_name}" type="rgbd_camera">
+      <sensor name="${prefix}${camera_name}" type="depth">
+        <plugin name="${prefix}${camera_name}_plugin" filename="libgazebo_ros_camera.so">
+          <ros>
+            <namespace>${prefix}</namespace>
+            <remapping>~/out:=${camera_name}</remapping>
+          </ros>
+          <camera_name>${camera_name}</camera_name>
+          <frame_name>${prefix}${camera_name}_depth_optical_frame</frame_name>
+          <hack_baseline>0.07</hack_baseline>
+          <min_depth>${clip_near}</min_depth>
+          <max_depth>${clip_far}</max_depth>
+        </plugin>
         <camera>
           <horizontal_fov>${horizontal_fov}</horizontal_fov>
@@ -131,4 +142,5 @@
             <width>${image_width}</width>
             <height>${image_height}</height>
+            <format>R8G8B8</format>
           </image>
           <clip>
@@ -138,8 +150,7 @@
         </camera>
         <always_on>${always_on}</always_on>
-        <gz_frame_id>${prefix}${camera_name}_depth_optical_frame</gz_frame_id>
-        <topic>${camera_name}</topic>
         <update_rate>${update_rate}</update_rate>
         <visualize>${visualize}</visualize>
+        <gz_frame_id>${prefix}${camera_name}_depth_optical_frame</gz_frame_id>
       </sensor>
     </gazebo>
