Commit message: Add Gazebo Fortress simulation with physics-based mecanum drive
- New launch file: rosmaster_gazebo_fortress.launch.py using ros_gz_sim,
  gz_ros2_control, and ros_gz_bridge for Fortress 6 compatibility
- mecanum_wheel.urdf.xacro: sphere collision + gz:expressed_in="base_link"
  fdir1 locks friction direction to chassis frame for correct holonomic
  strafing; reduces wheel mass 0.15→0.05 kg; increases joint damping
- rosmaster_x3.urdf.xacro: conditional gz_ros2_control vs
  gazebo_ros2_control plugin based on use_ignition flag
- rosmaster_x3_ros2_control.urdf.xacro: conditional GazeboSimSystem vs
  GazeboSystem hardware plugin
- rosmaster_x3_base.urdf.xacro: chassis mass 4.6→1.5 kg (real robot)
- empty.world: rewritten for Fortress (DART physics, inline light/ground,
  explicit system plugins replacing model:// URIs)
- ros2_control.yaml: add use_sim_time, velocity/acceleration limits,
  corrected wheel_separation 0.169→0.149 m
- ros_gz_bridge.yaml: remove stale TwistStamped cmd_vel bridge entry
- README: document Fortress prerequisites, launch, controller verification,
  teleop keys, and physics notes

Co-Authored-By: Claude Sonnet 4.6 <noreply@anthropic.com>

File: yahboom_rosmaster_description/urdf/control/rosmaster_x3_ros2_control.urdf.xacro (robot description, xacro)
@@ -1,8 +1,13 @@
 <?xml version="1.0" ?>
 <robot xmlns:xacro="http://wiki.ros.org/xacro">
-    <xacro:macro name="yahboom_rosmaster_ros2_control" params="prefix use_gazebo">
+    <xacro:macro name="yahboom_rosmaster_ros2_control" params="prefix use_gazebo use_ignition:='false'">
         <ros2_control name="RobotSystem" type="system">
             <hardware>
-                <plugin>gazebo_ros2_control/GazeboSystem</plugin>
+                <xacro:if value="${use_ignition}">
+                    <plugin>gz_ros2_control/GazeboSimSystem</plugin>
+                </xacro:if>
+                <xacro:unless value="${use_ignition}">
+                    <plugin>gazebo_ros2_control/GazeboSystem</plugin>
+                </xacro:unless>
             </hardware>
             <joint name="${prefix}front_left_wheel_joint">

File: yahboom_rosmaster_description/urdf/mech/mecanum_wheel.urdf.xacro (robot description, xacro)
@@ -1,11 +1,11 @@
 <?xml version="1.0"?>
-<robot xmlns:xacro="http://www.ros.org/wiki/xacro">
+<robot xmlns:xacro="http://www.ros.org/wiki/xacro" xmlns:gz="http://gazebosim.org/schema">
   <xacro:property name="wheel_radius" value="0.0325" />
   <xacro:property name="wheel_separation" value="0.169" />
   <xacro:property name="wheel_width" value="0.03040" />
-  <xacro:property name="wheel_mass" value="0.15" />
+  <xacro:property name="wheel_mass" value="0.05" />  <!-- Real 65mm mecanum wheel ~40-60 g. Old 0.15 kg was 3× too heavy. -->
   <xacro:property name="wheel_xoff" value="0.08" />
   <xacro:property name="wheel_yoff" value="-0.01" />
-  <xacro:macro name="mecanum_wheel" params="prefix side x_reflect y_reflect">
+  <xacro:macro name="mecanum_wheel" params="prefix side x_reflect y_reflect fdir1:='1 0 0' use_ignition:='false'">
     <link name="${prefix}${side}_wheel_link">
       <visual>
@@ -18,10 +18,22 @@
         </material>
       </visual>
-      <collision>
-        <origin xyz="0 0 0" rpy="${pi/2} 0 0"/>
-        <geometry>
-          <cylinder radius="${wheel_radius}" length="${wheel_width}"/>
-        </geometry>
-      </collision>
+      <!-- Fortress: sphere gives a single contact point, required for gz:expressed_in to work -->
+      <xacro:if value="${use_ignition}">
+        <collision>
+          <origin xyz="0 0 0" rpy="0 0 0"/>
+          <geometry>
+            <sphere radius="${wheel_radius}"/>
+          </geometry>
+        </collision>
+      </xacro:if>
+      <!-- Classic: cylinder collision (unchanged) -->
+      <xacro:unless value="${use_ignition}">
+        <collision>
+          <origin xyz="0 0 0" rpy="${pi/2} 0 0"/>
+          <geometry>
+            <cylinder radius="${wheel_radius}" length="${wheel_width}"/>
+          </geometry>
+        </collision>
+      </xacro:unless>
       <inertial>
         <origin xyz="0 0 0" rpy="0 0 0"/>
@@ -38,5 +50,5 @@
       <child link="${prefix}${side}_wheel_link"/>
       <origin xyz="${x_reflect*wheel_xoff} ${y_reflect*(wheel_separation/2+wheel_yoff)} ${-wheel_radius}" rpy="0 0 0"/>
-      <dynamics damping="0.01" friction="0.0"/>
+      <dynamics damping="0.1" friction="0.0"/>  <!-- 0.1 N·m·s/rad models 520-motor gearbox back-drive resistance -->
     </joint>
     <gazebo reference="${prefix}${side}_wheel_link">
@@ -45,6 +57,11 @@
           <ode>
               <mu>1.0</mu>
-              <mu2>0.5</mu2>
-              <fdir1>1 0 0</fdir1>
+              <mu2>0.0</mu2>
+              <xacro:if value="${use_ignition}">
+                <fdir1 gz:expressed_in="${prefix}base_link">${fdir1}</fdir1>
+              </xacro:if>
+              <xacro:unless value="${use_ignition}">
+                <fdir1>${fdir1}</fdir1>
+              </xacro:unless>
           </ode>
         </friction>

File: yahboom_rosmaster_description/urdf/mech/rosmaster_x3_base.urdf.xacro (robot description, xacro)
@@ -11,5 +11,5 @@
 <xacro:property name="base_size_y" value="${total_width - (2 * wheel_width)}" />
 <xacro:property name="base_size_z" value="${total_height - (2 * wheel_radius)}" />
-<xacro:property name="base_mass" value="4.6" />
+<xacro:property name="base_mass" value="1.5" />  <!-- Real X3: ~1.3 kg chassis+motors+PCBs + ~0.2 kg SBC/mount. Old value 4.6 kg was ~3× too heavy. -->
 <xacro:macro name="rosmaster_x3_base" params="prefix">
   <link name="${prefix}base_footprint"/>

File: yahboom_rosmaster_description/urdf/robots/rosmaster_x3.urdf.xacro (robot description, xacro)
@@ -1,8 +1,9 @@
 <?xml version="1.0"?>
-<robot xmlns:xacro="http://www.ros.org/wiki/xacro" name="rosmaster_x3">
+<robot xmlns:xacro="http://www.ros.org/wiki/xacro" xmlns:gz="http://gazebosim.org/schema" name="rosmaster_x3">
   <xacro:property name="M_PI" value="3.1415926535897931" />
   <xacro:arg name="robot_name" default="rosmaster_x3"/>
   <xacro:arg name="prefix" default=""/>
   <xacro:arg name="use_gazebo" default="false"/>
+  <xacro:arg name="use_ignition" default="false"/>
   <xacro:include filename="$(find yahboom_rosmaster_description)/urdf/mech/rosmaster_x3_base.urdf.xacro"/>
   <xacro:include filename="$(find yahboom_rosmaster_description)/urdf/mech/mecanum_wheel.urdf.xacro"/>
@@ -15,25 +16,33 @@
     side="front_left"
     x_reflect="1"
-    y_reflect="1"/>
+    y_reflect="1"
+    fdir1="1 -1 0"
+    use_ignition="$(arg use_ignition)"/>
   <xacro:mecanum_wheel
     prefix="$(arg prefix)"
     side="front_right"
     x_reflect="1"
-    y_reflect="-1"/>
+    y_reflect="-1"
+    fdir1="1 1 0"
+    use_ignition="$(arg use_ignition)"/>
   <xacro:mecanum_wheel
     prefix="$(arg prefix)"
     side="back_left"
     x_reflect="-1"
-    y_reflect="1"/>
+    y_reflect="1"
+    fdir1="1 1 0"
+    use_ignition="$(arg use_ignition)"/>
   <xacro:mecanum_wheel
     prefix="$(arg prefix)"
     side="back_right"
     x_reflect="-1"
-    y_reflect="-1"/>
+    y_reflect="-1"
+    fdir1="1 -1 0"
+    use_ignition="$(arg use_ignition)"/>
   <xacro:rgbd_camera
     prefix="$(arg prefix)"
     camera_name="cam_1"
     xyz_offset="0.105 0 0.05"
-    rpy_offset="0 -0.50 0"/>
+    rpy_offset="0 0 0"/>
   <xacro:lidar_sensor
     prefix="$(arg prefix)"
@@ -53,11 +62,20 @@
     update_rate="15.0"
     topic_name="imu/data"/>
-  <!-- Gazebo Classic ros2_control plugin -->
+  <!-- Gazebo ros2_control plugin — Fortress (gz_ros2_control) or Classic (gazebo_ros2_control) -->
   <xacro:if value="$(arg use_gazebo)">
-    <gazebo>
-      <plugin name="gazebo_ros2_control" filename="libgazebo_ros2_control.so">
-        <parameters>$(find yahboom_rosmaster_gazebo)/config/ros2_control.yaml</parameters>
-      </plugin>
-    </gazebo>
+    <xacro:if value="$(arg use_ignition)">
+      <gazebo>
+        <plugin filename="gz_ros2_control-system" name="gz_ros2_control::GazeboSimROS2ControlPlugin">
+          <parameters>$(find yahboom_rosmaster_gazebo)/config/ros2_control.yaml</parameters>
+        </plugin>
+      </gazebo>
+    </xacro:if>
+    <xacro:unless value="$(arg use_ignition)">
+      <gazebo>
+        <plugin name="gazebo_ros2_control" filename="libgazebo_ros2_control.so">
+          <parameters>$(find yahboom_rosmaster_gazebo)/config/ros2_control.yaml</parameters>
+        </plugin>
+      </gazebo>
+    </xacro:unless>
   </xacro:if>
   <!-- ros2_control joints/interfaces for the robot -->
@@ -65,4 +83,5 @@
   <xacro:yahboom_rosmaster_ros2_control
     prefix="$(arg prefix)"
-    use_gazebo="$(arg use_gazebo)"/>
+    use_gazebo="$(arg use_gazebo)"
+    use_ignition="$(arg use_ignition)"/>
 </robot>

File: yahboom_rosmaster_description/urdf/sensors/imu.urdf.xacro (robot description, xacro)
@@ -20,4 +20,6 @@
         gazebo_material_specular:='0.1 0.1 0.1 1'
         update_rate:='15.0'
+        gyro_noise_stddev:='0.00873'
+        accel_noise_stddev:='0.00175'
         topic_name:='imu/data'
         always_on:=true
@@ -67,4 +69,16 @@
                     <initial_orientation_as_reference>false</initial_orientation_as_reference>
                 </plugin>
+                <imu>
+                    <angular_velocity>
+                        <x><noise type="gaussian"><mean>0</mean><stddev>${gyro_noise_stddev}</stddev></noise></x>
+                        <y><noise type="gaussian"><mean>0</mean><stddev>${gyro_noise_stddev}</stddev></noise></y>
+                        <z><noise type="gaussian"><mean>0</mean><stddev>${gyro_noise_stddev}</stddev></noise></z>
+                    </angular_velocity>
+                    <linear_acceleration>
+                        <x><noise type="gaussian"><mean>0</mean><stddev>${accel_noise_stddev}</stddev></noise></x>
+                        <y><noise type="gaussian"><mean>0</mean><stddev>${accel_noise_stddev}</stddev></noise></y>
+                        <z><noise type="gaussian"><mean>0</mean><stddev>${accel_noise_stddev}</stddev></noise></z>
+                    </linear_acceleration>
+                </imu>
                 <update_rate>${update_rate}</update_rate>
                 <always_on>${always_on}</always_on>

File: yahboom_rosmaster_description/urdf/sensors/lidar.urdf.xacro (robot description, xacro)
@@ -31,4 +31,6 @@
     max_range:='30.0'
     range_resolution:='0.013'
+    noise_mean:='0.0'
+    noise_stddev:='0.02'
     topic_name:='scan'
     always_on:=true
@@ -111,4 +113,9 @@
             <resolution>${range_resolution}</resolution>
           </range>
+          <noise>
+            <type>gaussian</type>
+            <mean>${noise_mean}</mean>
+            <stddev>${noise_stddev}</stddev>
+          </noise>
         </ray>
         <gz_frame_id>${prefix}${frame_id}</gz_frame_id>
