Commit message: Simulation up and running

File: yahboom_rosmaster_description/urdf/mech/mecanum_wheel.urdf.xacro (robot description, xacro)
@@ -4,5 +4,5 @@
   <xacro:property name="wheel_separation" value="0.169" />
   <xacro:property name="wheel_width" value="0.03040" />
-  <xacro:property name="wheel_mass" value="0.4" />
+  <xacro:property name="wheel_mass" value="9.1" />
   <xacro:property name="wheel_xoff" value="0.08" />
   <xacro:property name="wheel_yoff" value="-0.01" />
@@ -21,5 +21,5 @@
         <origin xyz="0 0 0" rpy="${pi/2} 0 0"/>
         <geometry>
-          <sphere radius="${wheel_radius}"/>
+          <cylinder radius="${wheel_radius}" length="${wheel_width}"/>
         </geometry>
       </collision>
@@ -37,42 +37,24 @@
       <parent link="${prefix}base_link"/>
       <child link="${prefix}${side}_wheel_link"/>
-      <origin xyz="${x_reflect*wheel_xoff} ${y_reflect*(wheel_separation/2+wheel_yoff)} -0.003" rpy="0 0 0"/>
-      <limit effort="10.0" velocity="10.0"/>
+      <origin xyz="${x_reflect*wheel_xoff} ${y_reflect*(wheel_separation/2+wheel_yoff)} ${-wheel_radius}" rpy="0 0 0"/>
     </joint>
-    <!-- Add joint damping/friction to reduce drift at rest -->
-    <gazebo reference="${prefix}${side}_wheel_joint">
-      <dynamics damping="0.01" friction="0.0"/>
-    </gazebo>
-    <!-- Wheel contact/friction tuning for Gazebo Classic -->
-    <!-- Wheel contact/friction tuning for Gazebo Classic -->
     <gazebo reference="${prefix}${side}_wheel_link">
       <surface>
         <friction>
           <ode>
-            <mu>0.8</mu>
-            <mu2>0.8</mu2>
-            <fdir1>1 0 0</fdir1>
-            <slip1>0.0</slip1>
-            <slip2>0.0</slip2>
+              <mu>1.0</mu>
+              <mu2>0.0</mu2>
           </ode>
         </friction>
-        <contact>
-          <ode>
-            <kp>1000000.0</kp>
-            <kd>100.0</kd>
-            <max_vel>0.1</max_vel>
-            <min_depth>0.001</min_depth>
-          </ode>
-        </contact>
       </surface>
       <visual>
-        <material>
-          <ambient>0.2 0.2 0.2 1.0</ambient>
-          <diffuse>0.2 0.2 0.2 1.0</diffuse>
-          <specular>0.2 0.2 0.2 1.0</specular>
-          <emissive>0.0 0.0 0.0 0.0</emissive>
-        </material>
+          <material>
+              <ambient>0.2 0.2 0.2 1.0</ambient>
+              <diffuse>0.2 0.2 0.2 1.0</diffuse>
+              <specular>0.2 0.2 0.2 1.0</specular>
+              <emissive>0.0 0.0 0.0 0.0</emissive>
+          </material>
       </visual>
-    </gazebo>
+  </gazebo>
   </xacro:macro>
 </robot>

File: yahboom_rosmaster_description/urdf/robots/rosmaster_x3.urdf.xacro (robot description, xacro)
@@ -60,4 +60,19 @@
       </plugin>
     </gazebo>
+    <!-- Planar move plugin for holonomic/mecanum movement -->
+    <gazebo>
+      <plugin name="object_controller" filename="libgazebo_ros_planar_move.so">
+        <ros>
+          <remapping>cmd_vel:=mecanum_drive_controller/reference_unstamped</remapping>
+          <remapping>odom:=mecanum_drive_controller/odom</remapping>
+        </ros>
+        <update_rate>100</update_rate>
+        <publish_rate>10</publish_rate>
+        <publish_odom>true</publish_odom>
+        <publish_odom_tf>true</publish_odom_tf>
+        <odometry_frame>odom</odometry_frame>
+        <robot_base_frame>base_footprint</robot_base_frame>
+      </plugin>
+    </gazebo>
   </xacro:if>
   <!-- ros2_control joints/interfaces for the robot -->

Commit message: Added real physics working with gazebo engine. Deep testing still needed.

File: yahboom_rosmaster_description/urdf/mech/mecanum_wheel.urdf.xacro (robot description, xacro)
@@ -4,5 +4,5 @@
   <xacro:property name="wheel_separation" value="0.169" />
   <xacro:property name="wheel_width" value="0.03040" />
-  <xacro:property name="wheel_mass" value="9.1" />
+  <xacro:property name="wheel_mass" value="0.15" />
   <xacro:property name="wheel_xoff" value="0.08" />
   <xacro:property name="wheel_yoff" value="-0.01" />
@@ -38,4 +38,5 @@
       <child link="${prefix}${side}_wheel_link"/>
       <origin xyz="${x_reflect*wheel_xoff} ${y_reflect*(wheel_separation/2+wheel_yoff)} ${-wheel_radius}" rpy="0 0 0"/>
+      <dynamics damping="0.01" friction="0.0"/>
     </joint>
     <gazebo reference="${prefix}${side}_wheel_link">
@@ -44,7 +45,15 @@
           <ode>
               <mu>1.0</mu>
-              <mu2>0.0</mu2>
+              <mu2>0.5</mu2>
+              <fdir1>1 0 0</fdir1>
           </ode>
         </friction>
+        <contact>
+          <ode>
+            <kp>1000000.0</kp>
+            <kd>100.0</kd>
+            <min_depth>0.001</min_depth>
+          </ode>
+        </contact>
       </surface>
       <visual>

File: yahboom_rosmaster_description/urdf/robots/rosmaster_x3.urdf.xacro (robot description, xacro)
@@ -60,19 +60,4 @@
       </plugin>
     </gazebo>
-    <!-- Planar move plugin for holonomic/mecanum movement -->
-    <gazebo>
-      <plugin name="object_controller" filename="libgazebo_ros_planar_move.so">
-        <ros>
-          <remapping>cmd_vel:=mecanum_drive_controller/reference_unstamped</remapping>
-          <remapping>odom:=mecanum_drive_controller/odom</remapping>
-        </ros>
-        <update_rate>100</update_rate>
-        <publish_rate>10</publish_rate>
-        <publish_odom>true</publish_odom>
-        <publish_odom_tf>true</publish_odom_tf>
-        <odometry_frame>odom</odometry_frame>
-        <robot_base_frame>base_footprint</robot_base_frame>
-      </plugin>
-    </gazebo>
   </xacro:if>
   <!-- ros2_control joints/interfaces for the robot -->
